File: bkm-129x-simple.kicad_pcb (KiCad board)
At the start: 2 copper layers, 105 x 89.3 mm, 55 parts, among them J1 YG1, J2 PBB1, J3 PRR1, J4 SYNC1, J5 Conn_02x32_Row_Letter_Last, Q1 DTC144EKA, U1 ADG1611, U2 THS7374, U3 arduino-nano-v3, U4 74LVC125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

Commit message: Rev. D: THS7374 LPF, Kicad 5
Connections:
- U2 pad 9: GND -> +3V3
Routing:
- net GND: track 10.9 -> 9.63 mm, vias 8 -> 7
- net +3V3: track 29.0 -> 29.6 mm
Other:
- rule pad_to_mask_clearance: 0.2 -> 0
- board text added: "Rev. D"
- board text removed: "Rev. C"
